File: ESP8266_12E_breakout/ESP8266_12E_breakout.sch (KiCad schematic (older format))
At the start: 17 parts

Commit message: completed layout for breakout
Parts:
- removed D? (x2): LED, symbol LED
- removed J?: CONN_01X06, symbol CONN_01X06
- removed Q? (x2): BC547, TO_SOT_Packages_THT:TO-92_Molded_Narrow, symbol BC547
- removed R? (x2): 100, symbol R
- C1: renamed from C?; footprint (none) -> Capacitors_THT:CP_Radial_D5.0mm_P2.50mm
- C2: renamed from C?; footprint (none) -> Capacitors_THT:C_Disc_D3.0mm_W1.6mm_P2.50mm
- J2, J3: renamed from J?; footprint (none) -> Pin_Headers:Pin_Header_Straight_1x08_Pitch2.54mm
- R1, R2, R3, R4, R5: renamed from R?; footprint (none) -> Resistors_THT:R_Axial_DIN0207_L6.3mm_D2.5mm_P7.62mm_Horizontal
- U1: renamed from U?; footprint (none) -> ESP8266:ESP-12E_SMD
Connections:
- net labels removed: VCC
- wire segments 55 -> 37
