File: ESP8266_12E_breakout/_autosave-ESP8266_12E_breakout.kicad_pcb (KiCad board)
At the start: 2 copper layers, 10 parts, among them J2 CONN_01X08, J3 CONN_01X08, U1 ESP-12E

Commit message: completed layout for breakout
Changed lines of the file:
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@@
     (mod_text_size 1 1)
     (mod_text_width 0.15)
-    (pad_size 1.8 1.8)
-    (pad_drill 0.762)
+    (pad_size 1.7 2)
+    (pad_drill 1)
     (pad_to_mask_clearance 0.2)
     (aux_axis_origin 0 0)
@@
       (outputformat 1)
       (mirror false)
-      (drillshape 1)
+      (drillshape 0)
       (scaleselection 1)
       (outputdirectory ""))
@@
     (pad 5 thru_hole oval (at 0 10.16 180) (size 1.7 1.7) (drill 1) (layers *.Cu *.Mask)
       (net 7 /GPIO16))
-    (pad 4 thru_hole oval (at 0 7.62 180) (size 1.7 1.7) (drill 1) (layers *.Cu *.Mask)
+    (pad 4 thru_hole oval (at 0 7.62 180) (size 1.7 2) (drill 1) (layers *.Cu *.Mask)
       (net 8 /GPIO14))
     (pad 3 thru_hole oval (at 0 5.08 180) (size 1.7 1.7) (drill 1) (layers *.Cu *.Mask)
